File: board/board.kicad_pcb (KiCad board)
At the start: 4 copper layers, 219 parts, among them J1 USB_B_Micro, J2 USB_B_Micro, J3 Conn_01x30, J5 Conn_01x30, J7 Conn_01x02, J8 Conn_01x02, Q1 Q_PMOS_GSD, Q10 Q_NMOS_GSD, Q11 Q_PMOS_GSD, Q12 Q_NMOS_GSD, Q13 Q_PMOS_GSD, Q14 Q_NMOS_GSD, Q15 Q_PMOS_GSD, Q16 Q_NMOS_GSD, Q17 Q_PMOS_GSD, Q18 Q_NMOS_GSD, Q19 Q_PMOS_GSD, Q2 Q_NMOS_GSD, Q20 Q_NMOS_GSD, Q21 Q_PMOS_GSD, Q22 Q_NMOS_GSD, Q23 Q_PMOS_GSD, Q24 Q_NMOS_GSD, Q25 Q_PMOS_GSD, Q26 Q_NMOS_GSD, Q27 Q_PMOS_GSD, Q28 Q_NMOS_GSD, Q29 Q_PMOS_GSD, Q3 Q_PMOS_GSD, Q30 Q_NMOS_GSD, Q31 Q_PMOS_GSD, Q32 Q_NMOS_GSD, Q33 Q_PMOS_GSD, Q34 Q_NMOS_GSD, Q35 Q_PMOS_GSD, Q36 Q_NMOS_GSD, Q37 Q_PMOS_GSD, Q38 Q_NMOS_GSD, Q39 Q_PMOS_GSD, Q4 Q_NMOS_GSD, Q40 Q_NMOS_GSD, Q41 Q_PMOS_GSD, Q42 Q_NMOS_GSD, Q43 Q_PMOS_GSD, Q44 Q_NMOS_GSD, Q45 Q_PMOS_GSD, Q46 Q_NMOS_GSD, Q47 Q_PMOS_GSD, Q48 Q_NMOS_GSD, Q49 Q_PMOS_GSD, Q5 Q_PMOS_GSD, Q50 Q_NMOS_GSD, Q51 Q_PMOS_GSD, Q52 Q_NMOS_GSD, Q53 Q_PMOS_GSD, Q54 Q_NMOS_GSD, Q55 Q_PMOS_GSD, Q56 Q_NMOS_GSD, Q57 Q_PMOS_GSD, Q58 Q_NMOS_GSD, Q59 Q_PMOS_GSD, Q6 Q_NMOS_GSD, Q60 Q_NMOS_GSD, Q61 Q_PMOS_GSD, Q62 Q_NMOS_GSD, Q63 Q_PMOS_GSD, Q64 Q_NMOS_GSD, Q7 Q_PMOS_GSD, Q8 Q_NMOS_GSD, Q9 Q_PMOS_GSD, SW1 SW_Omron_B3FS, U1 93CxxC, U10 LM321, U11 LM321, U12 RP2040, U13 TXS0108EPW, U14 CD74HC4067M, U15 CD74HC4067M, U16 74HC595, U17 LM2901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

Commit message: More work before submitting
Parts:
- added J4: Conn_02x06_Odd_Even, Connector_PinHeader_2.54mm:PinHeader_2x06_P2.54mm_Horizontal, F.Cu at (129.6, 37.0)
- added R62: 10k, Resistor_SMD:R_0402_1005Metric, F.Cu at (134.7, 128.1)
- added R63: 10k, Resistor_SMD:R_0402_1005Metric, F.Cu at (81.3, 130.6)
- C12, C13: footprint Capacitor_SMD:C_0805_2012Metric -> Capacitor_SMD:C_0603_1608Metric
- C14, C15, C9: value 22u -> 10u
- R10, R18: value 30k -> 49.9k
- R11, R19: value 50k -> 49.9k
- U6, U8, U9: footprint 000_custom:SOT65P280X145-8N -> Package_TO_SOT_SMD:SOT-23-8
- moved C15 238.9 mm to (80.3, 141.1), turned to 180 degrees
- moved C13 232.1 mm to (76.6, 125.4), turned to 180 degrees
- moved R17 224.5 mm to (83.1, 134.0), turned to 90 degrees
- moved R19 223.5 mm to (80.2, 135.5), turned to 180 degrees
- moved FB2 218.6 mm to (80.3, 125.5)
- moved R22 217.9 mm to (81.8, 135.9), turned to -90 degrees
- moved R23 217.4 mm to (80.2, 136.5), turned to 180 degrees
- moved R11 216.6 mm to (79.3, 130.6)
- moved R15 215.4 mm to (84.6, 132.7), turned to -90 degrees
- moved R13 212.5 mm to (83.1, 132.0), turned to -90 degrees
- moved U7 207.2 mm to (80.3, 128.2), turned to 180 degrees
- moved U11 203.5 mm to (80.2, 133.1)
- moved U8 202.9 mm to (75.9, 128.1), turned to 180 degrees
- moved C14 195.0 mm to (125.2, 141.3), turned to 180 degrees
- moved L2 193.9 mm to (84.8, 128.7), turned to -90 degrees
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Connections:
- U12 pad 11: /PWR_B_DIN -> /PWR_A_DIN
- U12 pad 12: /PWR_B_~{CS} -> /PWR_A_~{CS}
- U12 pad 26: /RUN -> +3V3
- U12 pad 34: /GPIO22 -> /LCD_SCK
- U12 pad 35: /GPIO23 -> /LCD_MOSI
- U12 pad 36: /GPIO24 -> /LCD_MISO
- U12 pad 37: /GPIO25 -> /LCD_CS
- U12 pad 6: /PWR_A_SCLK -> /PWR_B_SCLK
- U12 pad 7: /PWR_A_DIN -> /PWR_B_DIN
- U12 pad 8: /PWR_A_~{CS} -> /PWR_B_~{CS}
- U12 pad 9: /PWR_B_SCLK -> /PWR_A_SCLK
Routing:
- net +3V3: track 0.00 -> 218.2 mm, vias 0 -> 24
- net /PWR_A: track 112.3 -> 290.0 mm, vias 16 -> 33
- net /CURRENT_SENSE_A: track 0.00 -> 126.0 mm, vias 0 -> 4
- net GND: track 189.1 -> 311.1 mm, vias 84 -> 108
- net /CURRENT_SENSE_B: track 0.00 -> 108.7 mm, vias 0 -> 4
- net /PWR_B_~{CS}: track 0.00 -> 103.4 mm, vias 0 -> 2
- net /PWR_A_SCLK: track 0.00 -> 101.6 mm, vias 0 -> 4
- net /PWR_B_DIN: track 0.00 -> 100.5 mm, vias 0 -> 2
- net /PWR_A_~{CS}: track 0.00 -> 98.4 mm, vias 0 -> 4
- net /PWR_A_DIN: track 0.00 -> 98.1 mm, vias 0 -> 4
- net /PWR_B_SCLK: track 0.00 -> 97.6 mm, vias 0 -> 4
- net VBUS: track 47.8 -> 135.7 mm, vias 25 -> 39
- net /PWR_B: track 87.8 -> 10.7 mm
- net /PIN_SENSE0: track 0.00 -> 43.1 mm, vias 0 -> 2
- net /FTDI_1V8: track 0.00 -> 35.1 mm
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- added copper zone on In2.Cu, net +3V3
Other:
- board outline added: 95 x 113 mm
- board text added: "3V3 CLK MOSI MISO ~{CS} GND"
- board text added: "Peter Schmidt-Nielsen https://peter.website"
