File: board/board.kicad_sch (KiCad schematic)
At the start: 77 parts, among them J1 USB_B_Micro, J2 USB_B_Micro, J3 Conn_01x30, J5 Conn_01x30, J7 Conn_01x02, J8 Conn_01x02, SW1 SW_Omron_B3FS, U1 93CxxC, U10 LM321, U11 LM321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

Commit message: More work before submitting
Parts:
- added J4: Conn_02x06_Odd_Even, Connector_PinHeader_2.54mm:PinHeader_2x06_P2.54mm_Horizontal, symbol Connector_Generic:Conn_02x06_Odd_Even
- C10, C11: LCSC (none) -> C1548
- C12, C13: footprint Capacitor_SMD:C_0805_2012Metric -> Capacitor_SMD:C_0603_1608Metric; LCSC (none) -> C1705
- C14, C15, C9: value 22u -> 10u; LCSC (none) -> C1713
- C16, C17: LCSC (none) -> C14445
- FB1, FB2: LCSC (none) -> C668237
- J2: LCSC (none) -> C428495
- J3, J5, J7, J8: now not fitted
- L1, L2: LCSC (none) -> C2929416
- R10, R18: value 30k -> 49.9k; LCSC (none) -> C25897
- R11, R19: value 50k -> 49.9k; LCSC (none) -> C25897
- R12, R13, R16, R17, R8, R9: LCSC (none) -> C11702
- R14, R15: LCSC (none) -> C474291
- R20, R22, R62, R63: LCSC (none) -> C25744
- R21, R23: LCSC (none) -> C25756
- R24, R25: LCSC (none) -> C25100
- R26, R28: LCSC (none) -> C25741
- R27, R29: LCSC (none) -> C25755
- SW1: LCSC (none) -> C493038
- U12: LCSC (none) -> C2040
- U13: LCSC (none) -> C17206
- U14, U15: LCSC (none) -> C496123
- U3: LCSC (none) -> C26537
- U4: LCSC (none) -> C97521
- U5, U7: LCSC (none) -> C398370
- U6, U8, U9: footprint 000_custom:SOT65P280X145-8N -> Package_TO_SOT_SMD:SOT-23-8; LCSC (none) -> C131323
- Y2: LCSC (none) -> C70565
Connections:
- net RUN is gone; now on net +3V3: U12.26 (RUN)
- net +3V3: now also J4.1 (Pin_1)
- net GND: now also J4.11 (Pin_11)
- net PWR_A_DIN: now also U12.11 (GPIO8); no longer U12.7 (GPIO5)
- net PWR_A_SCLK: now also U12.9 (GPIO7); no longer U12.6 (GPIO4)
- net PWR_A_~{CS}: now also U12.12 (GPIO9); no longer U12.8 (GPIO6)
- net PWR_B_DIN: now also U12.7 (GPIO5); no longer U12.11 (GPIO8)
- net PWR_B_SCLK: now also U12.6 (GPIO4); no longer U12.9 (GPIO7)
- net PWR_B_~{CS}: now also U12.8 (GPIO6); no longer U12.12 (GPIO9)
- net GPIO22 renamed LCD_SCK
- net LCD_SCK: now also J4.3 (Pin_3)
- net GPIO23 renamed LCD_MOSI
- net LCD_MOSI: now also J4.5 (Pin_5)
- net GPIO24 renamed LCD_MISO
- net LCD_MISO: now also J4.7 (Pin_7)
- net GPIO25 renamed LCD_CS
- net LCD_CS: now also J4.9 (Pin_9)
- no-connect marks 56 -> 62
