File: board/pin_group.kicad_sch (KiCad schematic)
At the start: 18 parts, among them Q1 Q_PMOS_GSD, Q2 Q_NMOS_GSD, Q3 Q_PMOS_GSD, Q4 Q_NMOS_GSD, Q5 Q_PMOS_GSD, Q6 Q_NMOS_GSD, Q7 Q_PMOS_GSD, Q8 Q_NMOS_GSD, U17 LM2901, U18 74HC595

Commit message: More work before submitting
Parts:
- R31, R32, R33, R34: LCSC (none) -> C11702
- U17: LCSC (none) -> C7932
- U18: LCSC (none) -> C431479
Changed lines of the file:
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@@
+			)
+		)
+		(property "LCSC" "C7932"
+			(at 144.145 126.365 0)
+			(effects
+				(font
+					(size 1.27 1.27)
+				)
+				(hide yes)
 			)
 		)
@@
 			)
 		)
+		(property "LCSC" "C7932"
+			(at 103.505 104.775 0)
+			(effects
+				(font
+					(size 1.27 1.27)
+				)
+				(hide yes)
+			)
+		)
 		(pin "8"
 		)
@@
 			)
 		)
+		(property "LCSC" "C11702"
+			(at 160.655 99.695 0)
+			(effects
+				(font
+					(size 1.27 1.27)
+				)
+				(hide yes)
+			)
+		)
 		(pin "1"
 		)
@@
 		)
 		(property "Description" "Resistor"
+			(at 160.655 126.365 0)
+			(effects
+				(font
+					(size 1.27 1.27)
+				)
+				(hide yes)
+			)
+		)
+		(property "LCSC" "C11702"
 			(at 160.655 126.365 0)
 			(effects
@@
 			)
 		)
+		(property "LCSC" "C7932"
+			(at 144.145 112.395 0)
+			(effects
+				(font
+					(size 1.27 1.27)
+				)
+				(hide yes)
+			)
+		)
 		(pin "8"
 		)
@@
 			)
 		)
+		(property "LCSC" "C7932"
+			(at 144.145 85.725 0)
+			(effects
+				(font
+					(size 1.27 1.27)
+				)
+				(hide yes)
+			)
+		)
 		(pin "8"
 		)
@@
 			)
 		)
+		(property "LCSC" "C7932"
+			(at 144.145 99.695 0)
+			(effects
+				(font
+					(size 1.27 1.27)
+				)
+				(hide yes)
+			)
+		)
 		(pin "8"
 		)
@@
 			)
 		)
+		(property "LCSC" "C431479"
+			(at 54.61 102.87 0)
+			(effects
+				(font
+					(size 1.27 1.27)
+				)
+				(hide yes)
+			)
+		)
 		(pin "5"
 		)
@@
 		)
 		(property "Description" "Resistor"
+			(at 160.655 112.395 0)
+			(effects
+				(font
+					(size 1.27 1.27)
+				)
+				(hide yes)
+			)
+		)
+		(property "LCSC" "C11702"
 			(at 160.655 112.395 0)
 			(effects
@@
 			(at 160.655 85.725 0)
 			(effects
+				(font
+					(size 1.27 1.27)
+				)
+				(hide yes)
+			)
+		)
+		(property "LCSC" "C11702"
+			(at 160.655 85.725 0)
+			(effects
